File: eagle/Receiver/Receiver.sch (EAGLE design)
At the start: 6 parts, among them IC1 ATMEGA325P

Commit message: Updating receiver to include wifi and ftdi.
Parts:
- added D1: U57X32, led:U57X32
- added IC2: FT230XS, ftdichip:FT230XS
- added R1: (no value), resistor:R-US_0204/5
- added U$1: NRF24L01, nrf24l01:NRF24L01
Connections:
- new net N$1: D1.A, IC1.CLKO/PCINT7/PE7
- new net N$11: IC1.OC0A/PCINT12/PB4, U$1.MISO
- new net N$13: IC1.RXD/PCINT0/PE0, IC2.TXD
- new net N$2: IC1.SCK/PCINT9/PB1, U$1.CE
- new net N$5: D1.C, R1.2
- new net N$6: IC1.MOSI/PCINT10/PB2, U$1.CSN
- new net N$7: IC1.OC1A/PCINT13/PB5, U$1.SCK
- new net N$8: IC1.MISO/PCINT11/PB3, U$1.MOSI
- new net N$9: IC1.TXD/PCINT1/PE1, IC2.!RTS
- net GND: now also IC2.GND, IC2.GND@1, R1.1
- net VCC: now also IC2.VCC
Changed lines of the file:
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@@
 <part name="GND1" library="supply1" deviceset="GND" device=""/>
 <part name="GND8" library="supply1" deviceset="GND" device=""/>
+<part name="GND4" library="supply1" deviceset="GND" device=""/>
+<part name="D1" library="led" deviceset="U57X32" device=""/>
+<part name="R1" library="resistor" deviceset="R-US_" device="0204/5"/>
+<part name="GND6" library="supply1" deviceset="GND" device=""/>
+<part name="IC2" library="ftdichip" deviceset="FT230X" device="S"/>
+<part name="U$1" library="nrf24l01" deviceset="NRF24L01" device=""/>
+<part name="GND5" library="supply1" deviceset="GND" device=""/>
+<part name="GND7" library="supply1" deviceset="GND" device=""/>
+<part name="P+5" library="supply1" deviceset="VCC" device=""/>
 </parts>
 <sheets>
@@
 <instance part="GND1" gate="1" x="93.98" y="5.08"/>
 <instance part="GND8" gate="1" x="83.82" y="27.94"/>
+<instance part="GND4" gate="1" x="134.62" y="-2.54"/>
+<instance part="D1" gate="1" x="27.94" y="66.04" rot="R270"/>
+<instance part="R1" gate="G$1" x="15.24" y="66.04"/>
+<instance part="GND6" gate="1" x="2.54" y="66.04" rot="R270"/>
+<instance part="IC2" gate="G$1" x="17.78" y="99.06" rot="R180"/>
+<instance part="U$1" gate="G$1" x="12.7" y="27.94"/>
+<instance part="GND5" gate="1" x="-5.08" y="99.06" rot="R270"/>
+<instance part="GND7" gate="1" x="40.64" y="101.6" rot="R90"/>
+<instance part="P+5" gate="VCC" x="-5.08" y="106.68" rot="R90"/>
 </instances>
 <busses>
@@
 </net>
 <net name="GND" class="0">
-<segment>
-<pinref part="R2" gate="G$1" pin="2"/>
-<wire x1="134.62" y1="2.54" x2="134.62" y2="0" width="0.1524" layer="91"/>
-</segment>
 <segment>
 <pinref part="GND2" gate="1" pin="GND"/>
@@
 <wire x1="101.6" y1="101.6" x2="101.6" y2="96.52" width="0.1524" layer="91"/>
 </segment>
-</net>
-<net name="N$16" class="0">
-<segment>
-<wire x1="25.4" y1="106.68" x2="63.5" y2="106.68" width="0.1524" layer="91"/>
-<wire x1="63.5" y1="106.68" x2="63.5" y2="111.76" width="0.1524" layer="91"/>
+<segment>
+<pinref part="R2" gate="G$1" pin="2"/>
+<pinref part="GND4" gate="1" pin="GND"/>
+<wire x1="134.62" y1="2.54" x2="134.62" y2="0" width="0.1524" layer="91"/>
+</segment>
+<segment>
+<pinref part="GND6" gate="1" pin="GND"/>
+<pinref part="R1" gate="G$1" pin="1"/>
+<wire x1="5.08" y1="66.04" x2="10.16" y2="66.04" width="0.1524" layer="91"/>
+</segment>
+<segment>
+<pinref part="GND5" gate="1" pin="GND"/>
+<pinref part="IC2" gate="G$1" pin="GND@1"/>
+<wire x1="-2.54" y1="99.06" x2="2.54" y2="99.06" width="0.1524" layer="91"/>
+</segment>
+<segment>
+<pinref part="IC2" gate="G$1" pin="GND"/>
+<pinref part="GND7" gate="1" pin="GND"/>
+<wire x1="33.02" y1="101.6" x2="38.1" y2="101.6" width="0.1524" layer="91"/>
 </segment>
 </net>
@@
 <pinref part="IC1" gate="G$1" pin="VCC@1"/>
 <wire x1="104.14" y1="104.14" x2="104.14" y2="96.52" width="0.1524" layer="91"/>
+</segment>
+<segment>
+<pinref part="P+5" gate="VCC" pin="VCC"/>
+<wire x1="-2.54" y1="106.68" x2="0" y2="106.68" width="0.1524" layer="91"/>
+<wire x1="0" y1="106.68" x2="0" y2="101.6" width="0.1524" layer="91"/>
+<pinref part="IC2" gate="G$1" pin="VCC"/>
+<wire x1="0" y1="101.6" x2="2.54" y2="101.6" width="0.1524" layer="91"/>
 </segment>
 </net>
@@
 </segment>
 </net>
+<net name="N$5" class="0">
+<segment>
+<pinref part="R1" gate="G$1" pin="2"/>
+<pinref part="D1" gate="1" pin="C"/>
+<wire x1="20.32" y1="66.04" x2="22.86" y2="66.04" width="0.1524" layer="91"/>
+</segment>
+</net>
+<net name="N$1" class="0">
+<segment>
+<pinref part="D1" gate="1" pin="A"/>
+<pinref part="IC1" gate="G$1" pin="CLKO/PCINT7/PE7"/>
+<wire x1="30.48" y1="66.04" x2="45.72" y2="66.04" width="0.1524" layer="91"/>
+</segment>
+</net>
+<net name="N$2" class="0">
+<segment>
+<pinref part="U$1" gate="G$1" pin="CE"/>
+<wire x1="27.94" y1="22.86" x2="30.48" y2="22.86" width="0.1524" layer="91"/>
+<wire x1="30.48" y1="22.86" x2="30.48" y2="60.96" width="0.1524" layer="91"/>
+<wire x1="30.48" y1="60.96" x2="45.72" y2="60.96" width="0.1524" layer="91"/>
+<pinref part="IC1" gate="G$1" pin="SCK/PCINT9/PB1"/>
+</segment>
+</net>
+<net name="N$6" class="0">
+<segment>
+<pinref part="U$1" gate="G$1" pin="CSN"/>
+<wire x1="27.94" y1="20.32" x2="33.02" y2="20.32" width="0.1524" layer="91"/>
+<wire x1="33.02" y1="20.32" x2="33.02" y2="58.42" width="0.1524" layer="91"/>
+<wire x1="33.02" y1="58.42" x2="45.72" y2="58.42" width="0.1524" layer="91"/>
+<pinref part="IC1" gate="G$1" pin="MOSI/PCINT10/PB2"/>
+</segment>
+</net>
+<net name="N$7" class="0">
+<segment>
+<pinref part="U$1" gate="G$1" pin="SCK"/>
+<wire x1="27.94" y1="17.78" x2="43.18" y2="17.78" width="0.1524" layer="91"/>
+<wire x1="43.18" y1="17.78" x2="43.18" y2="48.26" width="0.1524" layer="91"/>
+<wire x1="43.18" y1="48.26" x2="45.72" y2="48.26" width="0.1524" layer="91"/>
+<pinref part="IC1" gate="G$1" pin="OC1A/PCINT13/PB5"/>
+</segment>
+</net>
+<net name="N$8" class="0">
+<segment>
+<wire x1="45.72" y1="55.88" x2="35.56" y2="55.88" width="0.1524" layer="91"/>
+<wire x1="35.56" y1="55.88" x2="35.56" y2="15.24" width="0.1524" layer="91"/>
+<pinref part="U$1" gate="G$1" pin="MOSI"/>
+<wire x1="35.56" y1="15.24" x2="27.94" y2="15.24" width="0.1524" layer="91"/>
+<pinref part="IC1" gate="G$1" pin="MISO/PCINT11/PB3"/>
+</segment>
+</net>
+<net name="N$11" class="0">
+<segment>
+<pinref part="U$1" gate="G$1" pin="MISO"/>
+<wire x1="27.94" y1="12.7" x2="38.1" y2="12.7" width="0.1524" layer="91"/>
+<wire x1="38.1" y1="12.7" x2="38.1" y2="53.34" width="0.1524" layer="91"/>
+<wire x1="38.1" y1="53.34" x2="45.72" y2="53.34" width="0.1524" layer="91"/>
+<pinref part="IC1" gate="G$1" pin="OC0A/PCINT12/PB4"/>
+</segment>
+</net>
+<net name="N$9" class="0">
+<segment>
+<pinref part="IC2" gate="G$1" pin="!RTS"/>
+<wire x1="33.02" y1="93.98" x2="40.64" y2="93.98" width="0.1524" layer="91"/>
+<wire x1="40.64" y1="93.98" x2="40.64" y2="81.28" width="0.1524" layer="91"/>
+<pinref part="IC1" gate="G$1" pin="TXD/PCINT1/PE1"/>
+<wire x1="40.64" y1="81.28" x2="45.72" y2="81.28" width="0.1524" layer="91"/>
+</segment>
+</net>
+<net name="N$13" class="0">
+<segment>
+<pinref part="IC2" gate="G$1" pin="TXD"/>
+<wire x1="33.02" y1="91.44" x2="38.1" y2="91.44" width="0.1524" layer="91"/>
+<wire x1="38.1" y1="91.44" x2="38.1" y2="83.82" width="0.1524" layer="91"/>
+<pinref part="IC1" gate="G$1" pin="RXD/PCINT0/PE0"/>
+<wire x1="38.1" y1="83.82" x2="45.72" y2="83.82" width="0.1524" layer="91"/>
+</segment>
+</net>
